Commit message: Add URDF printer simulation to the G-code preview

File: assets/Pentos_URDF/urdf/Pentos_URDF.urdf (robot description, URDF)
Before this commit: robot Pentos_URDF, 6 links, 5 joints
Links:
- added link nozzle_tip
- added link plate_center
Joints:
- added joint nozzle_tip_joint: type fixed, parent x_carriage_link, child nozzle_tip, origin xyz=0 0 0 rpy=0 0 0
- added joint plate_center_joint: type fixed, parent b_rotary_link, child plate_center, origin xyz=0 0 0.05363390981229364 rpy=0 0 0
- joint b_joint: axis 0.00321170129672137 0 -0.99999484247409 -> 0 0 -1
- joint x_joint: limit lower=0 upper=0.22 effort=100 velocity=0.1 -> lower=-0.1154051200585088 upper=0.1045948799414912 effort=100 velocity=0.1; origin xyz=0.281542895629293 0.012908398513512 -0.0342499999998885 rpy=0 0 0 -> xyz=0.1661377755707842 0.012908398513512 -0.0342499999998885 rpy=0 0 0
- joint y_joint: limit lower=0 upper=0.15 effort=100 velocity=0.1 -> lower=-0.03792051833939079 upper=0.1120794816606092 effort=100 velocity=0.1; origin xyz=3.33215954637254E-05 -0.0257794816606062 0.16840013399872 rpy=0 0 0 -> xyz=3.33215954637254e-05 -0.063699999999997 0.16840013399872 rpy=0 0 0
- joint z_joint: limit lower=0 upper=0.19 effort=100 velocity=0.02 -> lower=0.0004937791330254793 upper=0.1904937791330255 effort=100 velocity=0.02; origin xyz=0.166342895629293 -0.0507916014864869 0.203286678805914 rpy=0 0 3.14159265358979 -> xyz=0.166342895629293 -0.0507916014864869 0.2027928996728885 rpy=0 0 3.14159265358979
